Commit message: (feat) Updated Ergo Jr meshes

File: simulator/ergo_jr/ergo_jr.urdf (robot description, URDF)
Before this commit: robot poppy_ergo_jr, 8 links, 7 joints
Links:
- removed link fixed_tip
- removed link section_5
- added link tip, mass 0.0164859649700598; collision mesh filename=package://meshes/tip.STL; visual mesh filename=package://meshes/tip.STL
- link base_link: mass None -> 0.0802410895423366; geometry collision mesh filename=package://meshes/base_link.STL; visual mesh filename=package://meshes/base_link.STL
- link long_U: mass 0.1 -> 0.0042118228619085; geometry collision mesh filename=package://meshes/long_U.STL; visual mesh filename=package://meshes/long_U.STL
- link section_1: mass 0.1 -> 0.0201321844066136; geometry collision mesh filename=package://meshes/section_1.STL; visual mesh filename=package://meshes/section_1.STL
- link section_2: mass 0.1 -> 0.017821725151696; geometry collision mesh filename=package://meshes/section_2.STL; visual mesh filename=package://meshes/section_2.STL
- link section_3: mass 0.1 -> 0.0201321844066136; geometry collision mesh filename=package://meshes/section_3.STL; visual mesh filename=package://meshes/section_3.STL
- link section_4: mass 0.1 -> 0.0201321844066137; geometry collision mesh filename=package://meshes/section_4.STL; visual mesh filename=package://meshes/section_4.STL
Joints:
- removed joint t7f
- joint m1: axis 0 0 1 -> 0 0 -1; origin xyz=0 0 0.0327993216120967 rpy=0 0 0 -> xyz=0 0 0.0327993216120967 rpy=-6.12303176911189E-17 0 0
- joint m2: axis 0 0 -1 -> -1 0 0; origin xyz=0 0 0.0240006783879033 rpy=0 -1.5707963267949 0 -> xyz=0 0 0.0240006783879033 rpy=1.5707963267949 0 0
- joint m3: axis 0 0 -1 -> -1 0 0; origin xyz=0.054 0 0 rpy=0 0 0 -> xyz=0 0.054 0 rpy=0 0 0
- joint m4: axis 0 0 -1 -> 0 1 0; origin xyz=0.045 0 0 rpy=0 -1.5707963267949 0 -> xyz=0 0.0298217741221248 0 rpy=3.14159265358979 0 0
- joint m5: axis 0 0 1 -> -1 0 0; origin xyz=0 -0.048 0 rpy=0 -1.5707963267949 0 -> xyz=0 -0.0151782258778753 -0.048 rpy=-1.5707963267949 0 0
- joint m6: axis 0 0 1 -> 0 -1 0; child section_5 -> tip; origin xyz=0 -0.054 0 rpy=0 0 0 -> xyz=0 0.054 0 rpy=1.5707963267949 1.5707963267949 0

Commit message: (feat) Working inverse kinematics simulation

File: simulator/ergo_jr/ergo_jr.urdf (robot description, URDF)
Before this commit: robot PoppyErgoJr, 7 links, 6 joints
Joints:
- joint m1: type continuous -> revolute
- joint m2: type continuous -> revolute
- joint m3: type continuous -> revolute
- joint m4: type continuous -> revolute
- joint m5: type continuous -> revolute
- joint m6: type continuous -> revolute
